Commit message: Re #11: Added logic to parse urdf for stl file name. Updated file names in launch omni as well. Unsure about if we should use relative path or not.

File: models/urdf/omni.urdf (robot description, URDF)
Before this commit: robot phantom_omni, 7 links, 6 joints
Links:
- link base: geometry visual mesh filename=/ros2_ws/src/SlicerRos2/models/meshes/base.stl
- link lower_arm: geometry visual mesh filename=/ros2_ws/src/SlicerRos2/models/meshes/lower_arm.stl
- link stylus: geometry visual mesh filename=/ros2_ws/src/SlicerRos2/models/meshes/pen.stl
- link tip: geometry visual mesh filename=/ros2_ws/src/SlicerRos2/models/meshes/tip.stl
- link torso: geometry visual mesh filename=/ros2_ws/src/SlicerRos2/models/meshes/torso.stl
- link upper_arm: geometry visual mesh filename=/ros2_ws/src/SlicerRos2/models/meshes/upper_arm.stl
- link wrist: geometry visual mesh filename=/ros2_ws/src/SlicerRos2/models/meshes/wrist.stl
